Commit message: :bug: [Fix] robot 실측값으로 통일

File: ros/WSL/src/robot_description/urdf/robot.urdf.xacro (robot description, xacro)
@@ -10,5 +10,5 @@
   <xacro:property name="wheel_radius"      value="0.033"/>  <!-- 바퀴 반지름 33mm -->
   <xacro:property name="wheel_width"       value="0.025"/>  <!-- 바퀴 폭 25mm (추정) -->
-  <xacro:property name="wheel_separation"  value="0.100"/>  <!-- 좌우 바퀴 중심 간격 230mm (실측 220~240, 중간값) -->
+  <xacro:property name="wheel_separation"  value="0.100"/>  <!-- 좌우 바퀴 중심 간격 100mm (실측) -->
   <!-- base_link 원점 = 로봇 중심, 지면에서 wheel_radius 높이 -->
   <xacro:property name="base_z_offset"     value="${wheel_radius}"/>

Commit message: :bug: [Fix] stm32와 sync 맞추기

File: ros/WSL/src/robot_description/urdf/robot.urdf.xacro (robot description, xacro)
@@ -8,7 +8,7 @@
   <xacro:property name="base_width"        value="0.140"/>  <!-- 좌우 140mm -->
   <xacro:property name="base_height"       value="0.200"/>  <!-- 플레이트 두께 60mm (추정) -->
-  <xacro:property name="wheel_radius"      value="0.033"/>  <!-- 바퀴 반지름 33mm -->
+  <xacro:property name="wheel_radius"      value="0.0325"/> <!-- 바퀴 반지름 32.5mm (65mm 지름 실측) -->
   <xacro:property name="wheel_width"       value="0.025"/>  <!-- 바퀴 폭 25mm (추정) -->
-  <xacro:property name="wheel_separation"  value="0.100"/>  <!-- 좌우 바퀴 중심 간격 100mm (실측) -->
+  <xacro:property name="wheel_separation"  value="0.230"/>  <!-- 좌우 바퀴 중심 간격 230mm (실측) -->
   <!-- base_link 원점 = 로봇 중심, 지면에서 wheel_radius 높이 -->
   <xacro:property name="base_z_offset"     value="${wheel_radius}"/>

Commit message: :bug: [Fix] wheel_base 수정

File: ros/WSL/src/robot_description/urdf/robot.urdf.xacro (robot description, xacro)
@@ -10,5 +10,5 @@
   <xacro:property name="wheel_radius"      value="0.0325"/> <!-- 바퀴 반지름 32.5mm (65mm 지름 실측) -->
   <xacro:property name="wheel_width"       value="0.025"/>  <!-- 바퀴 폭 25mm (추정) -->
-  <xacro:property name="wheel_separation"  value="0.230"/>  <!-- 좌우 바퀴 중심 간격 230mm (실측) -->
+  <xacro:property name="wheel_separation"  value="0.100"/>  <!-- 좌우 바퀴 중심 간격 100mm (실측) -->
   <!-- base_link 원점 = 로봇 중심, 지면에서 wheel_radius 높이 -->
   <xacro:property name="base_z_offset"     value="${wheel_radius}"/>

Commit message: :bug: [Fix] 실측값 수정

File: ros/WSL/src/robot_description/urdf/robot.urdf.xacro (robot description, xacro)
@@ -8,5 +8,5 @@
   <xacro:property name="base_width"        value="0.140"/>  <!-- 좌우 140mm -->
   <xacro:property name="base_height"       value="0.200"/>  <!-- 플레이트 두께 60mm (추정) -->
-  <xacro:property name="wheel_radius"      value="0.0325"/> <!-- 바퀴 반지름 32.5mm (65mm 지름 실측) -->
+  <xacro:property name="wheel_radius"      value="0.0329"/> <!-- 바퀴 반지름 32.9mm (serial_bridge 캘리브레이션 값과 통일) -->
   <xacro:property name="wheel_width"       value="0.025"/>  <!-- 바퀴 폭 25mm (추정) -->
   <xacro:property name="wheel_separation"  value="0.100"/>  <!-- 좌우 바퀴 중심 간격 100mm (실측) -->
